File: indicateur_batterie_v1/indicateur_batterie_v1.kicad_sch (KiCad schematic)
At the start: 13 parts, among them J1 Conn_01x02_Pin, Q1 Q_PMOS_GSD, U1 ATtiny412-SS, U3 MCP1802x-xx02xOT

Commit message: changement déclanchement télécomande
Parts:
- D3: value D_Schottky -> BAT54W D_Schottky
Changed lines of the file:
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@@
 			)
 		)
-		(property "Value" "D_Schottky"
+		(property "Value" "BAT54W D_Schottky"
 			(at 49.8475 54.61 0)
 			(effects
